File: hardware/yacobo-blue.kicad_pcb (KiCad board)
At the start: 2 copper layers, 150 x 38 mm, 15 parts, among them J1 USB_B, J2 columns, J3 rows, J4 leds, M1 MountingHole_3.5mm, M2 MountingHole_3.5mm, M3 MountingHole_3.5mm, M4 MountingHole_3.5mm, U1 STM32F103C8T6

Commit message: support 12 pin configuration
Parts:
- J3: footprint Connector_PinHeader_2.54mm:PinHeader_1x08_P2.54mm_Vertical -> Connector_PinHeader_2.54mm:PinHeader_1x12_P2.54mm_Vertical
- U1: value STM32F103C8T6 -> BluePill_STM32F103C
- moved R4 10.6 mm to (228.0, 115.2)
- moved R3 10.4 mm to (228.0, 112.2)
- moved R5 10.3 mm to (228.0, 120.0)
- moved J4 6.50 mm to (243.5, 112.5)
Connections:
- J4 pad 1: Net-(J4-Pad1) -> Net-(J3-Pad12)
- J4 pad 2: Net-(J4-Pad2) -> Net-(J3-Pad11)
- J4 pad 4: Net-(J4-Pad4) -> Net-(J3-Pad9)
- R3 pad 2: Net-(J4-Pad1) -> Net-(J3-Pad12)
- R4 pad 2: Net-(J4-Pad2) -> Net-(J3-Pad11)
- R5 pad 2: Net-(J4-Pad4) -> Net-(J3-Pad9)
Routing:
- net Net-(J3-Pad9): track 0.00 -> 25.7 mm
- net Net-(J4-Pad2): track 19.6 -> 0.00 mm
- net Net-(J4-Pad1): track 19.1 -> 0.00 mm
- net Net-(J4-Pad4): track 19.0 -> 0.00 mm
- net +3V3: track 78.9 -> 95.2 mm
- net Net-(J3-Pad11): track 0.00 -> 16.1 mm
- net Net-(J3-Pad12): track 0.00 -> 11.8 mm
- net led1: track 44.6 -> 56.1 mm
- net led0: track 48.7 -> 60.0 mm
- net led2: track 40.5 -> 51.6 mm
Other:
- board text added: "Yacobo v1.1"
- board text removed: "v1.0"

Commit message: space out cols vs rows. Add 3v3 top fill version.
Routing:
- net col15: track 62.4 -> 61.1 mm
Other:
- net class Default removed
- net class Power removed
- board text added: "Yacobo v1.2"
- board text removed: "Yacobo v1.1"
